Commit message: first functional version of robot (showing robot odometry)

File: urdf/robotic_bird.urdf.xacro (robot description, xacro)
@@ -14,7 +14,19 @@
     </collision>
     <inertial>
-      <mass value="1.0"/>
-      <inertia ixx="0.1" iyy="0.1" izz="0.1" ixy="0.0" ixz="0.0" iyz="0.0"/>
+      <mass>5.0</mass>
+      <inertia>
+        <ixx>0.1</ixx> <ixy>0.0</ixy> <ixz>0.0</ixz>
+        <iyy>0.1</iyy> <iyz>0.0</iyz> <izz>0.1</izz>
+      </inertia>
     </inertial>
   </link>
+  <!-- Set dynamic properties -->
+  <gazebo reference="base_link">
+    <static>false</static>
+    <material>Gazebo/Blue</material>
+  </gazebo>
+  <!-- Single plugin configuration -->
+  <gazebo>
+    <plugin name="flap_plugin" filename="libflap_plugin.so"/>
+  </gazebo>
 </robot>

Commit message: functional flight control (but not giving desired trajectory)

File: urdf/robotic_bird.urdf.xacro (robot description, xacro)
@@ -1,4 +1,5 @@
 <?xml version="1.0"?>
 <robot name="robotic_bird" xmlns:xacro="http://www.ros.org/wiki/xacro">
+  <!-- Base link -->
   <link name="base_link">
     <visual>
@@ -6,5 +7,7 @@
         <sphere radius="0.2"/>
       </geometry>
-      <material name="blue"/>
+      <material name="blue">
+        <color rgba="0 0 1 1"/>
+      </material>
     </visual>
     <collision>
@@ -14,19 +17,24 @@
     </collision>
     <inertial>
-      <mass>5.0</mass>
-      <inertia>
-        <ixx>0.1</ixx> <ixy>0.0</ixy> <ixz>0.0</ixz>
-        <iyy>0.1</iyy> <iyz>0.0</iyz> <izz>0.1</izz>
-      </inertia>
+      <mass value="5.0"/>
+      <inertia
+        ixx="0.05" ixy="0" ixz="0"
+        iyy="0.05" iyz="0"
+        izz="0.05"/>
     </inertial>
   </link>
-  <!-- Set dynamic properties -->
+  <!-- Gazebo-specific properties -->
   <gazebo reference="base_link">
-    <static>false</static>
     <material>Gazebo/Blue</material>
+    <gravity>true</gravity>
+    <mu1>0.2</mu1>
+    <mu2>0.2</mu2>
   </gazebo>
-  <!-- Single plugin configuration -->
+  <!-- Flap plugin -->
   <gazebo>
-    <plugin name="flap_plugin" filename="libflap_plugin.so"/>
+    <plugin name="flap_plugin" filename="libflap_plugin.so">
+      <link_name>base_link</link_name>
+      <update_rate>100</update_rate>
+    </plugin>
   </gazebo>
 </robot>

Commit message: functional control with tuned parameters

File: urdf/robotic_bird.urdf.xacro (robot description, xacro)
@@ -15,19 +15,28 @@
         <sphere radius="0.2"/>
       </geometry>
+      <surface>
+        <contact>
+          <collide_bitmask>0</collide_bitmask>
+        </contact>
+      </surface>
     </collision>
     <inertial>
       <mass value="5.0"/>
       <inertia
-        ixx="0.05" ixy="0" ixz="0"
-        iyy="0.05" iyz="0"
-        izz="0.05"/>
+        ixx="0.08" ixy="0" ixz="0"
+        iyy="0.08" iyz="0"
+        izz="0.08"/>
     </inertial>
   </link>
   <!-- Gazebo-specific properties -->
   <gazebo reference="base_link">
-    <material>Gazebo/Blue</material>
     <gravity>true</gravity>
+    <self_collide>false</self_collide>
+    <kinematic>false</kinematic>
     <mu1>0.2</mu1>
     <mu2>0.2</mu2>
+    <kp>100000</kp> <!-- contact stiffness -->
+    <kd>1.0</kd>    <!-- contact damping -->
+    <allow_free_motion>true</allow_free_motion>
   </gazebo>
   <!-- Flap plugin -->
