Commit message: implement a realisic bird model

File: robotic_bird.urdf (robot description, URDF)
Before this commit: robot robotic_bird, 1 links, 0 joints
Links:
- removed link base_link
- added link body_link, mass 5.0; collision cylinder length=1 radius=0.05; visual cylinder length=1 radius=0.05
- added link head_link, mass 0.5; collision sphere radius=0.1; visual sphere radius=0.1
- added link left_wing_link, mass 0.3; collision cylinder length=0.7 radius=0.05; visual cylinder length=0.7 radius=0.05
- added link right_wing_link, mass 0.3; collision cylinder length=0.7 radius=0.05; visual cylinder length=0.7 radius=0.05
Joints:
- added joint head_joint: type fixed, parent body_link, child head_link, origin xyz=0 0 0.6 rpy=0 0 0
- added joint left_wing_joint: type fixed, parent body_link, child left_wing_link, origin xyz=0 0.25 0 rpy=0 0 0
- added joint right_wing_joint: type fixed, parent body_link, child right_wing_link, origin xyz=0 -0.25 0 rpy=0 0 0

File: urdf/robotic_bird.urdf.xacro (robot description, xacro)
@@ -1,9 +1,9 @@
 <?xml version="1.0"?>
 <robot name="robotic_bird" xmlns:xacro="http://www.ros.org/wiki/xacro">
-  <!-- Base link -->
-  <link name="base_link">
+  <!-- ================= BODY ================= -->
+  <link name="body_link">
     <visual>
       <geometry>
-        <sphere radius="0.2"/>
+        <cylinder radius="0.05" length="1"/>
       </geometry>
       <material name="blue">
@@ -13,22 +13,95 @@
     <collision>
       <geometry>
-        <sphere radius="0.2"/>
+        <cylinder radius="0.05" length="1"/>
       </geometry>
-      <surface>
-        <contact>
-          <collide_bitmask>0</collide_bitmask>
-        </contact>
-      </surface>
     </collision>
     <inertial>
       <mass value="5.0"/>
-      <inertia
-        ixx="0.08" ixy="0" ixz="0"
-        iyy="0.08" iyz="0"
-        izz="0.08"/>
+      <inertia ixx="0.05" iyy="0.05" izz="0.05" ixy="0" ixz="0" iyz="0"/>
     </inertial>
   </link>
+  <!-- ================= HEAD ================= -->
+  <link name="head_link">
+    <visual>
+      <geometry>
+        <sphere radius="0.1"/>
+      </geometry>
+      <material name="blue">
+        <color rgba="0 0 1 1"/>
+      </material>
+    </visual>
+    <collision>
+      <geometry>
+        <sphere radius="0.1"/>
+      </geometry>
+    </collision>
+    <inertial>
+      <mass value="0.5"/>
+      <inertia ixx="0.001" iyy="0.001" izz="0.001" ixy="0" ixz="0" iyz="0"/>
+    </inertial>
+  </link>
+  <joint name="head_joint" type="fixed">
+    <parent link="body_link"/>
+    <child link="head_link"/>
+    <origin xyz="0 0 0.6" rpy="0 0 0"/>
+  </joint>
+  <!-- ================= LEFT WING ================= -->
+  <link name="left_wing_link">
+    <visual>
+      <!-- Rotate cylinder along Y-axis (wing span) -->
+      <origin xyz="0 0 0" rpy="0 0 1.5708"/>
+      <geometry>
+        <cylinder radius="0.05" length="0.7"/>
+      </geometry>
+      <material name="blue">
+        <color rgba="0 0 1 1"/>
+      </material>
+    </visual>
+    <collision>
+      <origin xyz="0 0 0" rpy="0 0 1.5708"/>
+      <geometry>
+        <cylinder radius="0.05" length="0.7"/>
+      </geometry>
+    </collision>
+    <inertial>
+      <mass value="0.3"/>
+      <inertia ixx="0.0005" iyy="0.0005" izz="0.0001" ixy="0" ixz="0" iyz="0"/>
+    </inertial>
+  </link>
+  <joint name="left_wing_joint" type="fixed">
+    <parent link="body_link"/>
+    <child link="left_wing_link"/>
+    <origin xyz="0 0.25 0" rpy="0 0 0"/>
+  </joint>
+  <!-- ================= RIGHT WING ================= -->
+  <link name="right_wing_link">
+    <visual>
+      <!-- Rotate cylinder along Y-axis (wing span) -->
+      <origin xyz="0 0 0" rpy="0 0 1.5708"/>
+      <geometry>
+        <cylinder radius="0.05" length="0.7"/>
+      </geometry>
+      <material name="blue">
+        <color rgba="0 0 1 1"/>
+      </material>
+    </visual>
+    <collision>
+      <origin xyz="0 0 0" rpy="0 0 1.5708"/>
+      <geometry>
+        <cylinder radius="0.05" length="0.7"/>
+      </geometry>
+    </collision>
+    <inertial>
+      <mass value="0.3"/>
+      <inertia ixx="0.0005" iyy="0.0005" izz="0.0001" ixy="0" ixz="0" iyz="0"/>
+    </inertial>
+  </link>
+  <joint name="right_wing_joint" type="fixed">
+    <parent link="body_link"/>
+    <child link="right_wing_link"/>
+    <origin xyz="0 -0.25 0" rpy="0 0 0"/>
+  </joint>
   <!-- Gazebo-specific properties -->
-  <gazebo reference="base_link">
+  <gazebo reference="body_link">
     <gravity>true</gravity>
     <self_collide>false</self_collide>
@@ -43,5 +116,5 @@
   <gazebo>
     <plugin name="flap_plugin" filename="libflap_plugin.so">
-      <link_name>base_link</link_name>
+      <link_name>body_link</link_name>
       <update_rate>100</update_rate>
     </plugin>
